File: egg58v2/egg58v2_switchplate.kicad_pcb (KiCad board)
At the start: 2 copper layers, 129 x 127.1 mm, 34 parts, among them SW11 SW_PUSH_LED, SW12 SW_PUSH_LED, SW13 SW_PUSH_LED, SW14 SW_PUSH_LED, SW15 SW_PUSH_LED, SW16 SW_PUSH_LED, SW21 SW_PUSH_LED, SW22 SW_PUSH_LED, SW23 SW_PUSH_LED, SW24 SW_PUSH_LED, SW25 SW_PUSH_LED, SW26 SW_PUSH_LED, SW31 SW_PUSH_LED, SW32 SW_PUSH_LED, SW33 SW_PUSH_LED, SW34 SW_PUSH_LED, SW35 SW_PUSH_LED, SW36 SW_PUSH_LED, SW41 SW_PUSH_LED, SW42 SW_PUSH_LED, SW43 SW_PUSH_LED, SW44 SW_PUSH_LED, SW45 SW_PUSH_LED, SW46 SW_PUSH_LED, SW52 SW_PUSH_LED, SW53 SW_PUSH_LED, SW54 SW_PUSH_LED, SW55 SW_PUSH_LED, SW56 SW_PUSH_LED

Commit message: Final touches on switchplate
Routing:
- added copper zone on B.Cu, net (none)
- added copper zone on F.Cu, net (none)
Other:
- board size 129 x 127.1 mm -> 128.5 x 127.1 mm
- board text added: "JLCJLCJLCJLC"
Changed lines of the file:
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@@
   (general
     (thickness 1.6)
-    (drawings 1)
+    (drawings 2)
     (tracks 0)
     (zones 0)
@@
     (pad 1 np_thru_hole circle (at 0 0) (size 2.2 2.2) (drill 2.2) (layers *.Cu *.Mask))
   )
-  (gr_poly (pts (xy 245 50) (xy 249 54) (xy 249 133.35) (xy 243.84 138.43) (xy 185.42 138.43) (xy 140.97 163.83) (xy 137.16 162.56) (xy 120.016362 133.490352) (xy 120.208793 132.688941) (xy 129.75 126.25) (xy 129.750159 39.750001) (xy 129.750191 39.75) (xy 130.247055 39.21294) (xy 161.25 36.75) (xy 209.88 37.5)) (layer Edge.Cuts) (width 0.1))
+  (gr_text JLCJLCJLCJLC (at 170.5 75.75 90) (layer F.SilkS)
+    (effects (font (size 1.5 1.5) (thickness 0.3)))
+  )
+  (gr_poly (pts (xy 245 50) (xy 249 54) (xy 249 133.35) (xy 243.84 138.43) (xy 185.42 138.43) (xy 140.97 163.83) (xy 137.16 162.56) (xy 120.473557 134.265595) (xy 120.955945 132.184721) (xy 129.75 126.25) (xy 129.750157 40.500001) (xy 130.992352 39.153732) (xy 161.25 36.75) (xy 209.88 37.5)) (layer Edge.Cuts) (width 0.1))
+  (zone (net 0) (net_name "") (layer F.Cu) (hatch edge 0.508)
+    (connect_pads (clearance 0.508))
+    (min_thickness 0.254)
+    (fill yes (arc_segments 32) (thermal_gap 0.508) (thermal_bridge_width 0.508))
+    (polygon
+      (pts
+        (xy 255 165.25) (xy 118.25 165.25) (xy 118.25 31) (xy 255 31)
+      )
+    )
+  )
+  (zone (net 0) (net_name "") (layer B.Cu) (hatch edge 0.508)
+    (connect_pads (clearance 0.508))
+    (min_thickness 0.254)
+    (fill yes (arc_segments 32) (thermal_gap 0.508) (thermal_bridge_width 0.508))
+    (polygon
+      (pts
+        (xy 255 31) (xy 254.75 165.5) (xy 118 165.75) (xy 118 30.75) (xy 118.25 30.75)
+      )
+    )
+  )
 )
