File: egg58v3/egg58v3-back.kicad_sch (KiCad schematic)
At the start: 29 parts, among them SW11 SW_PUSH_LED, SW12 SW_PUSH_LED, SW13 SW_PUSH_LED, SW14 SW_PUSH_LED, SW15 SW_PUSH_LED, SW16 SW_PUSH_LED, SW21 SW_PUSH_LED, SW22 SW_PUSH_LED, SW23 SW_PUSH_LED, SW24 SW_PUSH_LED, SW25 SW_PUSH_LED, SW26 SW_PUSH_LED, SW31 SW_PUSH_LED, SW32 SW_PUSH_LED, SW33 SW_PUSH_LED, SW34 SW_PUSH_LED, SW35 SW_PUSH_LED, SW36 SW_PUSH_LED, SW41 SW_PUSH_LED, SW42 SW_PUSH_LED, SW43 SW_PUSH_LED, SW44 SW_PUSH_LED, SW45 SW_PUSH_LED, SW46 SW_PUSH_LED, SW52 SW_PUSH_LED, SW53 SW_PUSH_LED, SW54 SW_PUSH_LED, SW55 SW_PUSH_LED, SW56 SW_PUSH_LED

Commit message: Initial layout for v3
Parts:
- SW55, SW56: footprint egg58v2:Choc_Hotswap_SK6812MiniE -> egg58v2:Choc_Hotswap_SK6812MiniE_Thumb
Changed lines of the file:
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@@
       (effects (font (size 0.635 0.635)) hide)
     )
-    (property "Footprint" "egg58v2:Choc_Hotswap_SK6812MiniE" (id 2) (at 130.81 128.778 0)
+    (property "Footprint" "egg58v2:Choc_Hotswap_SK6812MiniE_Thumb" (id 2) (at 130.81 128.778 0)
       (effects (font (size 1.27 1.27)) hide)
     )
@@
       (effects (font (size 0.635 0.635)) hide)
     )
-    (property "Footprint" "egg58v2:Choc_Hotswap_SK6812MiniE" (id 2) (at 226.822 124.46 0)
+    (property "Footprint" "egg58v2:Choc_Hotswap_SK6812MiniE_Thumb" (id 2) (at 226.822 124.46 0)
       (effects (font (size 1.27 1.27)) hide)
     )
@@
       (effects (font (size 0.635 0.635)) hide)
     )
-    (property "Footprint" "egg58v2:Choc_Hotswap_SK6812MiniE" (id 2) (at 113.03 128.778 0)
+    (property "Footprint" "egg58v2:Choc_Hotswap_SK6812MiniE_Thumb" (id 2) (at 113.03 128.778 0)
       (effects (font (size 1.27 1.27)) hide)
     )
@@
       (effects (font (size 0.635 0.635)) hide)
     )
-    (property "Footprint" "egg58v2:Choc_Hotswap_SK6812MiniE" (id 2) (at 126.492 120.65 0)
+    (property "Footprint" "egg58v2:Choc_Hotswap_SK6812MiniE_Thumb" (id 2) (at 126.492 120.65 0)
       (effects (font (size 1.27 1.27)) hide)
     )
@@
       (effects (font (size 0.635 0.635)) hide)
     )
-    (property "Footprint" "egg58v2:Choc_Hotswap_SK6812MiniE" (id 2) (at 144.272 120.65 0)
+    (property "Footprint" "egg58v2:Choc_Hotswap_SK6812MiniE_Thumb" (id 2) (at 144.272 120.65 0)
       (effects (font (size 1.27 1.27)) hide)
     )
@@
       (effects (font (size 0.635 0.635)) hide)
     )
-    (property "Footprint" "egg58v2:Choc_Hotswap_SK6812MiniE" (id 2) (at 239.522 114.3 0)
-      (effects (font (size 1.27 1.27)) hide)
-    )
+    (property "Footprint" "egg58v2:Choc_Hotswap_SK6812MiniE_Thumb" (id 2) (at 239.522 114.3 0)
+      (effects (font (size 1.27 1.27)) hide)
+    )
